Commit message: Adjusting Hector Mapping parameters

File: cartographer_config/backpack_2d.urdf (robot description, URDF)
Before this commit: robot cartographer_backpack_2d, 1 links, 0 joints
Links:
- added link base_laser, mass 10; collision box size=0.6 0.1 0.2; visual cylinder length=0.045 radius=0.036
- added link tf_tof_3_optical_frame, mass 10; collision box size=0.6 0.1 0.2; visual cylinder length=0.045 radius=0.036
- link base_link: mass None -> 10; geometry collision cylinder length=1 radius=0.50; visual box size=0.90 0.64 0.52
Joints:
- added joint base_to_laser: type fixed, parent base_link, child base_laser, origin xyz=0.20 -0.315 0.25 rpy=0 0 0
- added joint base_to_tf_front: type fixed, parent base_link, child tf_tof_3_optical_frame, origin xyz=0.20 0.315 0.25 rpy=0 0 0
